File: kicad/untitled.kicad_sch (KiCad schematic)
At the start: 26 parts, among them J1 PS2_USB, J2 Conn_01x08_Pin, J3 AVR-ISP-6, J4 Conn_01x04_Pin, J6 SD, J7 I2c, J8 LCD, SW2 SW_SPDT, U10 ATmega16A-P, U11 W65C22NxP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

Commit message: connect 6522 to simavr
Parts:
- U11: value W65C22NxP -> VIA0
- U15: value W65C22NxP -> VIA1
Changed lines of the file:
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@@
 			)
 		)
-		(property "Value" "W65C22NxP"
+		(property "Value" "VIA0"
 			(at 127.8733 53.34 0)
 			(show_name no)
@@
 			)
 		)
-		(property "Value" "W65C22NxP"
+		(property "Value" "VIA1"
 			(at 185.0233 80.01 0)
 			(show_name no)
