File: kicad/untitled.kicad_sch (KiCad schematic)
At the start: 26 parts, among them J1 PS2_USB, J2 Conn_01x08_Pin, J3 AVR-ISP-6, J4 Conn_01x04_Pin, J6 SD, J7 I2c, J8 LCD, SW2 SW_SPDT, U10 ATmega16A-P, U11 VIA0, U15 VIA1, Y2 16Mhz

Commit message: add third menu
Parts:
- added D1: 1N4148W, Diode_SMD:D_SOD-123, symbol Diode:1N4148W
- added H8: +5v, MountingHole:MountingHole_2.5mm_Pad_TopBottom, symbol Mechanical:MountingHole_Pad
- added H9: GND, MountingHole:MountingHole_2.5mm_Pad_TopBottom, symbol Mechanical:MountingHole_Pad
- added U6: SN74LVC126APWR-TP, Package_SO:TSSOP-14_4.4x5mm_P0.65mm, symbol 74xx:74LS126
Connections:
- net +3.3V: now also U6.14 (VCC)
- net +5V: now also J6.5 (Pin_5), J7.4 (Pin_4), H8.1, U6.1, U6.10, U6.13, U6.4; no longer J6.1 (Pin_1), J7.1 (Pin_1)
- net GND: now also H9.1, U6.7 (GND)
- net LCD_CK: now also U6.11
- net LCD_CS: now also U6.6
- net LCD_DC: now also U6.3
- net LCD_MOSI: now also U6.8
- net MOSI: now also U6.9
- net SCK: now also U6.12
- net SD_CS: now also J6.1 (Pin_1); no longer J6.5 (Pin_5)
- net ~{IRQ}: now also J7.1 (Pin_1); no longer J7.4 (Pin_4)
- net ~{RESET}: now also D1.2 (A); no longer J3.5 (~{RST}), U10.9 (~{RESET})
- net SDA: now reaches J7.3 (Pin_3), R4.1, U15.8 (PA6)
- net SCL: now reaches J7.2 (Pin_2), R3.1, U15.7 (PA5)
- net logicshift2/in: no longer names the net of U10.5 (PB4)
- net logicshift2/in: now also U6.5
- net logicshift3/in: no longer names the net of U10.4 (PB3)
- net logicshift3/in: now also U6.2
- new net ~{AVRRESET}: D1.1 (K), J3.5 (~{RST}), U10.9 (~{RESET})
Other:
- removed sheet logicshift
- removed sheet logicshift1
- removed sheet logicshift2
- removed sheet logicshift3
