File: kicad/osprey68.kicad_sch (KiCad schematic)
At the start: 11 parts, among them SW1 SW_Push, U1 MC6809E, U12 AMS1117-3.3, U2 74HC74, U5 GAL20V8, Y1 8Mhz

Commit message: add third menu
Parts:
- U2: footprint Package_DIP:DIP-14_W7.62mm_Socket -> Package_SO:SO-14_3.9x8.65mm_P1.27mm
Changed lines of the file:
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@@
 			)
 		)
-		(property "Footprint" "Package_DIP:DIP-14_W7.62mm_Socket"
+		(property "Footprint" "Package_SO:SO-14_3.9x8.65mm_P1.27mm"
 			(at 54.61 151.13 0)
 			(hide yes)
@@
 			)
 		)
-		(property "Footprint" "Package_DIP:DIP-14_W7.62mm_Socket"
+		(property "Footprint" "Package_SO:SO-14_3.9x8.65mm_P1.27mm"
 			(at 80.01 151.13 0)
 			(hide yes)
@@
 			)
 		)
-		(property "Footprint" "Package_DIP:DIP-14_W7.62mm_Socket"
+		(property "Footprint" "Package_SO:SO-14_3.9x8.65mm_P1.27mm"
 			(at 106.68 161.29 0)
 			(hide yes)
